File: board/board.kicad_pcb (KiCad board)
At the start: 2 copper layers, 21 x 13 mm, 1 part

Commit message: initial
Parts:
- added J1: 008_USB, on_edge:on_edge_2x05_device, F.Cu at (140.0, 97.0)
- added J2: USB_A, Connector_USB:USB_A_CONNFLY_DS1095-WNR0, F.Cu at (152.3, 103.5)
- added R1: 0R, Resistor_SMD:R_0603_1608Metric, F.Cu at (148.0, 93.0)
- moved LOGO1 10.0 mm to (146.5, 108.4)
Routing:
- net /usb-a/Schield: track 0.00 -> 19.5 mm
- net /usb-a/VUSB: track 0.00 -> 18.3 mm
- net /usb-a/DM: track 0.00 -> 11.4 mm
- net GND: track 0.00 -> 11.4 mm
- net /usb-a/DP: track 0.00 -> 11.3 mm
Other:
- board size 21 x 13 mm -> 21 x 29 mm
- board text added: "osf.008"
- board text added: "osf.b120.v1.0"
